Commit message: Structure visualization in RVIZ

File: robot_package/description/urdf/robot.urdf (robot description, URDF)
Before this commit: robot None, 4 links, 3 joints
Links:
- removed link caster_wheel
- added link bottom_edge, mass 5.0; visual box size=11.0 1.0 1.0
- added link left_column, mass 5.0; visual box size=1.0 1.0 17.5
- added link left_support, mass 5.0; visual box size=1.0 4.0 1.0
- added link right_column, mass 5.0; visual box size=1.0 1.0 17.5
- added link right_support, mass 5.0; visual box size=1.0 4.0 1.0
- added link support_left_wheel, mass 5.0; visual cylinder length=2.0 radius=0.25
- added link support_right_wheel, mass 5.0; visual cylinder length=2.0 radius=0.25
- added link top_edge, mass 5.0; visual box size=11.0 1.0 1.0
- added link whiteboard, mass 5.0; visual box size=10.0 0.5 10.0
- link base_link: mass 4.2 -> 5.0; geometry visual box size=1.0 0.5 1.0
- link left_wheel: mass 0.8 -> 5.0; geometry visual cylinder length=0.5 radius=0.5
- link right_wheel: mass 0.8 -> 5.0; geometry visual cylinder length=0.5 radius=0.5
Joints:
- removed joint connection_link
- added joint bottom_edge_joint: type fixed, parent base_link, child bottom_edge, origin xyz=5.0 0.0 7.0 rpy=0 0 0
- added joint left_column_joint: type fixed, parent base_link, child left_column, origin xyz=0.0 0.0 8.75 rpy=0 0 0
- added joint left_support_joint: type fixed, parent base_link, child left_support, origin xyz=0.0 0.0 0.5 rpy=0 0 0
- added joint right_column_joint: type fixed, parent base_link, child right_column, origin xyz=10.0 0.0 8.75 rpy=0 0 0
- added joint right_support_joint: type fixed, parent base_link, child right_support, origin xyz=10.0 0.0 0.5 rpy=0 0 0
- added joint support_left_wheel_joint: type fixed, parent base_link, child support_left_wheel, origin xyz=0.0 -0.5 17.0 rpy=-1.570796 0 0
- added joint support_right_wheel_joint: type fixed, parent base_link, child support_right_wheel, origin xyz=10.0 -0.5 17.0 rpy=-1.570796 0 0
- added joint top_edge_joint: type fixed, parent base_link, child top_edge, origin xyz=5.0 0.0 17.0 rpy=0 0 0
- added joint whiteboard_joint: type fixed, parent base_link, child whiteboard, origin xyz=5.0 0.0 12.0 rpy=0 0 0
- joint left_wheel_joint: origin xyz=-0.1 0.15 0.05 rpy=-1.570796 0 0 -> xyz=0.0 -1.25 17.0 rpy=-1.570796 0 0
- joint right_wheel_joint: origin xyz=-0.1 -0.15 0.05 rpy=-1.570796 0 0 -> xyz=10.0 -1.25 17.0 rpy=-1.570796 0 0

Commit message: Adding decimals

File: robot_package/description/urdf/robot.urdf (robot description, URDF)
Before this commit: robot None, 12 links, 11 joints
Joints:
- joint bottom_edge_joint: origin xyz=5.0 0.0 7.0 rpy=0 0 0 -> xyz=5.0 0.0 7.0 rpy=0.0 0.0 0.0
- joint left_column_joint: origin xyz=0.0 0.0 8.75 rpy=0 0 0 -> xyz=0.0 0.0 8.75 rpy=0.0 0.0 0.0
- joint left_support_joint: origin xyz=0.0 0.0 0.5 rpy=0 0 0 -> xyz=0.0 0.0 0.5 rpy=0.0 0.0 0.0
- joint left_wheel_joint: axis 0 0 1 -> 0.0 0.0 1.0; origin xyz=0.0 -1.25 17.0 rpy=-1.570796 0 0 -> xyz=0.0 -1.25 17.0 rpy=-1.570796 0.0 0.0
- joint right_column_joint: origin xyz=10.0 0.0 8.75 rpy=0 0 0 -> xyz=10.0 0.0 8.75 rpy=0.0 0.0 0.0
- joint right_support_joint: origin xyz=10.0 0.0 0.5 rpy=0 0 0 -> xyz=10.0 0.0 0.5 rpy=0.0 0.0 0.0
- joint right_wheel_joint: origin xyz=10.0 -1.25 17.0 rpy=-1.570796 0 0 -> xyz=10.0 -1.25 17.0 rpy=-1.570796 0.0 0.0
- joint support_left_wheel_joint: origin xyz=0.0 -0.5 17.0 rpy=-1.570796 0 0 -> xyz=0.0 -0.5 17.0 rpy=-1.570796 0.0 0.0
- joint support_right_wheel_joint: origin xyz=10.0 -0.5 17.0 rpy=-1.570796 0 0 -> xyz=10.0 -0.5 17.0 rpy=-1.570796 0.0 0.0
- joint top_edge_joint: origin xyz=5.0 0.0 17.0 rpy=0 0 0 -> xyz=5.0 0.0 17.0 rpy=0.0 0.0 0.0
- joint whiteboard_joint: origin xyz=5.0 0.0 12.0 rpy=0 0 0 -> xyz=5.0 0.0 12.0 rpy=0.0 0.0 0.0

Commit message: Cleaning urdf and TF tree

File: robot_package/description/urdf/robot.urdf (robot description, URDF)
Before this commit: robot None, 12 links, 11 joints
Links:
- added link end_effector, mass 5.00; visual box size=0.10 0.05 0.10
- link base_link: mass 5.0 -> None; geometry 
- link bottom_edge: mass 5.0 -> 5.00; geometry visual box size=1.10 0.10 0.10
- link left_column: mass 5.0 -> 5.00; geometry visual box size=0.10 0.10 1.75
- link left_support: mass 5.0 -> 5.00; geometry visual box size=0.10 0.40 0.10
- link left_wheel: mass 5.0 -> 5.00; geometry visual cylinder length=0.05 radius=0.05
- link right_column: mass 5.0 -> 5.00; geometry visual box size=0.10 0.10 1.75
- link right_support: mass 5.0 -> 5.00; geometry visual box size=0.10 0.40 0.10
- link right_wheel: mass 5.0 -> 5.00; geometry visual cylinder length=0.05 radius=0.05
- link support_left_wheel: mass 5.0 -> 5.00; geometry visual cylinder length=0.20 radius=0.025
- link support_right_wheel: mass 5.0 -> 5.00; geometry visual cylinder length=0.20 radius=0.025
- link top_edge: mass 5.0 -> 5.00; geometry visual box size=1.10 0.10 0.10
- link whiteboard: mass 5.0 -> 5.00; geometry visual box size=1.00 0.05 1.00
Joints:
- added joint end_effector_joint: type fixed, parent base_link, child end_effector, origin xyz=0.00 0.00 0.00 rpy=0.00 0.00 0.00
- joint bottom_edge_joint: origin xyz=5.0 0.0 7.0 rpy=0.0 0.0 0.0 -> xyz=0.50 0.00 0.70 rpy=0.00 0.00 0.00
- joint left_column_joint: origin xyz=0.0 0.0 8.75 rpy=0.0 0.0 0.0 -> xyz=0.00 0.00 0.875 rpy=0.00 0.00 0.00
- joint left_support_joint: origin xyz=0.0 0.0 0.5 rpy=0.0 0.0 0.0 -> xyz=0.00 0.00 0.05 rpy=0.00 0.00 0.00
- joint left_wheel_joint: axis 0.0 0.0 1.0 -> 0.00 0.00 1.00; origin xyz=0.0 -1.25 17.0 rpy=-1.570796 0.0 0.0 -> xyz=0.00 -0.125 1.70 rpy=-1.57 0.00 0.00
- joint right_column_joint: origin xyz=10.0 0.0 8.75 rpy=0.0 0.0 0.0 -> xyz=1.00 0.00 0.875 rpy=0.00 0.00 0.00
- joint right_support_joint: origin xyz=10.0 0.0 0.5 rpy=0.0 0.0 0.0 -> xyz=1.00 0.00 0.05 rpy=0.00 0.00 0.00
- joint right_wheel_joint: axis 0 0 1 -> 0.00 0.00 1.00; origin xyz=10.0 -1.25 17.0 rpy=-1.570796 0.0 0.0 -> xyz=1.00 -0.125 1.70 rpy=-1.57 0.00 0.00
- joint support_left_wheel_joint: origin xyz=0.0 -0.5 17.0 rpy=-1.570796 0.0 0.0 -> xyz=0.00 -0.05 1.70 rpy=-1.57 0.00 0.00
- joint support_right_wheel_joint: origin xyz=10.0 -0.5 17.0 rpy=-1.570796 0.0 0.0 -> xyz=1.00 -0.05 1.70 rpy=-1.57 0.00 0.00
- joint top_edge_joint: origin xyz=5.0 0.0 17.0 rpy=0.0 0.0 0.0 -> xyz=0.50 0.00 1.70 rpy=0.00 0.00 0.00
- joint whiteboard_joint: origin xyz=5.0 0.0 12.0 rpy=0.0 0.0 0.0 -> xyz=0.50 0.00 1.20 rpy=0.00 0.00 0.00
